File: files/w12-reflect.brd (EAGLE design)
At the start: 100 x 80 mm, 9 parts

Commit message: traces and outline png
Parts:
- moved C1 2.70 mm to (27.7, 5.33)
- moved R1 2.70 mm to (23.6, 5.33)
- moved R3 2.70 mm to (6.10, 15.7)
- moved U$1 2.70 mm to (17.5, 5.84)
- moved U$2 2.70 mm to (15.0, 15.7)
- moved U$4 2.70 mm to (6.10, 5.84)
- moved U$5 2.70 mm to (20.3, 15.7)
- moved R2 2.70 mm to (6.10, 13.0)
- moved U$3 2.70 mm to (33.0, 8.38)
Other:
- board size 100 x 80 mm -> 38.1 x 19.6 mm
