File: files/w14/controller.sch (EAGLE design)
At the start: 19 parts

Commit message: routing in progress
Parts:
- added IC2: 5V, fab:REGULATORSOT23
- added U$2: PINHD-2X2-SMD, fab:PINHD-2X2-SMD
Connections:
- new net VIN: IC2.IN, U$2.2
- net GND: now also IC2.GND, U$2.4; no longer U$3.GND
- net VCC: now also IC2.OUT; no longer U$3.VCC
Changed lines of the file:
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@@
 <parts>
 <part name="U$1" library="fab" deviceset="AVRISP" device="SMD"/>
+<part name="IC2" library="fab" deviceset="REGULATOR" device="SOT23" value="5V"/>
+<part name="U$2" library="fab" deviceset="PINHD-2X2-SMD" device=""/>
 <part name="U$17" library="fab" deviceset="ATTINY45" device="SI"/>
 <part name="R16" library="fab" deviceset="RES-US" device="1206FAB"/>
@@
 <instances>
 <instance part="U$1" gate="G$1" x="-5.08" y="55.88"/>
+<instance part="IC2" gate="G$1" x="60.96" y="106.68"/>
+<instance part="U$2" gate="G$1" x="15.24" y="109.22"/>
 <instance part="U$17" gate="G$1" x="81.28" y="81.28"/>
 <instance part="R16" gate="G$1" x="5.08" y="86.36"/>
@@
 </segment>
 <segment>
+<pinref part="IC2" gate="G$1" pin="OUT"/>
+<wire x1="68.58" y1="109.22" x2="78.74" y2="109.22" width="0.1524" layer="91"/>
+<label x="73.66" y="109.22" size="1.778" layer="95"/>
+</segment>
+<segment>
 <pinref part="U$17" gate="G$1" pin="VCC"/>
 <wire x1="116.84" y1="86.36" x2="132.08" y2="86.36" width="0.1524" layer="91"/>
@@
 <pinref part="C1" gate="&gt;NAME" pin="2"/>
 </segment>
-<segment>
-<pinref part="U$3" gate="G$1" pin="VCC"/>
-<wire x1="93.98" y1="106.68" x2="86.36" y2="106.68" width="0.1524" layer="91"/>
-<label x="86.36" y="106.68" size="1.778" layer="95"/>
-</segment>
 </net>
 <net name="GND" class="0">
@@
 <wire x1="0" y1="53.34" x2="12.7" y2="53.34" width="0.1524" layer="91"/>
 <label x="7.62" y="53.34" size="1.778" layer="95"/>
+</segment>
+<segment>
+<pinref part="IC2" gate="G$1" pin="GND"/>
+<wire x1="60.96" y1="104.14" x2="60.96" y2="96.52" width="0.1524" layer="91"/>
+<label x="60.96" y="96.52" size="1.778" layer="95"/>
+</segment>
+<segment>
+<pinref part="U$2" gate="G$1" pin="4"/>
+<wire x1="17.78" y1="109.22" x2="33.02" y2="109.22" width="0.1524" layer="91"/>
+<label x="27.94" y="109.22" size="1.778" layer="95"/>
 </segment>
 <segment>
@@
 <label x="-25.4" y="86.36" size="1.778" layer="95"/>
 </segment>
+</net>
+<net name="VIN" class="0">
 <segment>
-<pinref part="U$3" gate="G$1" pin="GND"/>
-<wire x1="93.98" y1="111.76" x2="86.36" y2="111.76" width="0.1524" layer="91"/>
-<label x="86.36" y="111.76" size="1.778" layer="95"/>
+<pinref part="U$2" gate="G$1" pin="2"/>
+<wire x1="17.78" y1="111.76" x2="33.02" y2="111.76" width="0.1524" layer="91"/>
+<label x="27.94" y="111.76" size="1.778" layer="95"/>
+</segment>
+<segment>
+<pinref part="IC2" gate="G$1" pin="IN"/>
+<wire x1="53.34" y1="109.22" x2="43.18" y2="109.22" width="0.1524" layer="91"/>
+<label x="43.18" y="109.22" size="1.778" layer="95"/>
 </segment>
 </net>
