File: files/w20/7-segment.sch (EAGLE design)
At the start: 18 parts

Commit message: 7segment board refactoring
Parts:
- removed R1, R2: (no value), fab:RES-US1206FAB
- removed U$3: FTDI-SMD-HEADER, fab:FTDI-SMD-HEADER
- added U$1: AVRISPSMD, fab:AVRISPSMD
Connections:
- net GND: now also U$1.GND; no longer U$3.GND
- net MISO: now also U$1.MISO; no longer U$3.RXD
- net MOSI: now also U$1.MOSI; no longer U$3.RTS
- net PB3: no longer R2.1, R2.2
- net RST: now also U$1.RST; no longer U$3.CTS
- net SCK: now also U$1.SCK; no longer R1.1, R1.2, U$3.TXD
- net VCC: now also U$1.VCC; no longer U$3.VCC
Changed lines of the file:
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@@
 <part name="RG" library="fab" deviceset="RES-US" device="1206FAB"/>
 <part name="LG" library="fab" deviceset="LED" device="FAB1206"/>
-<part name="U$3" library="fab" deviceset="FTDI-SMD-HEADER" device=""/>
-<part name="R1" library="fab" deviceset="RES-US" device="1206FAB"/>
-<part name="R2" library="fab" deviceset="RES-US" device="1206FAB"/>
+<part name="U$1" library="fab" deviceset="AVRISP" device="SMD"/>
 </parts>
 <sheets>
@@
 <instance part="RG" gate="G$1" x="114.3" y="137.16" rot="R270"/>
 <instance part="LG" gate="G$1" x="114.3" y="121.92"/>
-<instance part="U$3" gate="G$1" x="71.12" y="58.42" rot="R270"/>
-<instance part="R1" gate="G$1" x="7.62" y="83.82"/>
-<instance part="R2" gate="G$1" x="-7.62" y="127"/>
+<instance part="U$1" gate="G$1" x="43.18" y="50.8"/>
 </instances>
 <busses>
@@
 </segment>
 <segment>
-<pinref part="U$3" gate="G$1" pin="VCC"/>
-<wire x1="78.74" y1="58.42" x2="78.74" y2="66.04" width="0.1524" layer="91"/>
-<label x="78.74" y="66.04" size="1.778" layer="95" rot="R270"/>
+<pinref part="U$1" gate="G$1" pin="VCC"/>
+<wire x1="48.26" y1="53.34" x2="58.42" y2="53.34" width="0.1524" layer="91"/>
+<label x="53.34" y="53.34" size="1.778" layer="95"/>
 </segment>
 </net>
@@
 </segment>
 <segment>
-<pinref part="U$3" gate="G$1" pin="GND"/>
-<wire x1="83.82" y1="58.42" x2="83.82" y2="66.04" width="0.1524" layer="91"/>
-<label x="83.82" y="66.04" size="1.778" layer="95" rot="R270"/>
+<pinref part="U$1" gate="G$1" pin="GND"/>
+<wire x1="48.26" y1="48.26" x2="58.42" y2="48.26" width="0.1524" layer="91"/>
+<label x="53.34" y="48.26" size="1.778" layer="95"/>
 </segment>
 </net>
@@
 </segment>
 <segment>
-<pinref part="U$3" gate="G$1" pin="CTS"/>
-<wire x1="81.28" y1="58.42" x2="81.28" y2="66.04" width="0.1524" layer="91"/>
-<label x="81.28" y="66.04" size="1.778" layer="95" rot="R270"/>
+<pinref part="U$1" gate="G$1" pin="RST"/>
+<wire x1="40.64" y1="48.26" x2="30.48" y2="48.26" width="0.1524" layer="91"/>
+<label x="30.48" y="48.26" size="1.778" layer="95"/>
 </segment>
 </net>
@@
 <wire x1="33.02" y1="88.9" x2="17.78" y2="88.9" width="0.1524" layer="91"/>
 <label x="22.86" y="88.9" size="1.778" layer="95" rot="R180"/>
-</segment>
-<segment>
-<pinref part="U$3" gate="G$1" pin="RTS"/>
-<wire x1="71.12" y1="58.42" x2="71.12" y2="66.04" width="0.1524" layer="91"/>
-<label x="71.12" y="66.04" size="1.778" layer="95" rot="R270"/>
 </segment>
 <segment>
@@
 <junction x="91.44" y="147.32"/>
 </segment>
+<segment>
+<pinref part="U$1" gate="G$1" pin="MOSI"/>
+<wire x1="48.26" y1="50.8" x2="58.42" y2="50.8" width="0.1524" layer="91"/>
+<label x="53.34" y="50.8" size="1.778" layer="95"/>
+</segment>
 </net>
 <net name="MISO" class="0">
@@
 </segment>
 <segment>
-<pinref part="U$3" gate="G$1" pin="RXD"/>
-<wire x1="73.66" y1="58.42" x2="73.66" y2="66.04" width="0.1524" layer="91"/>
-<label x="73.66" y="66.04" size="1.778" layer="95" rot="R270"/>
+<pinref part="U$1" gate="G$1" pin="MISO"/>
+<wire x1="40.64" y1="53.34" x2="30.48" y2="53.34" width="0.1524" layer="91"/>
+<label x="30.48" y="53.34" size="1.778" layer="95"/>
 </segment>
 </net>
@@
 <segment>
 <pinref part="U$17" gate="G$1" pin="SCK/USCK/SCL/ADC1/T0/INT0/PCINT2/PB2"/>
-<wire x1="33.02" y1="83.82" x2="12.7" y2="83.82" width="0.1524" layer="91"/>
+<wire x1="33.02" y1="83.82" x2="17.78" y2="83.82" width="0.1524" layer="91"/>
 <label x="22.86" y="83.82" size="1.778" layer="95" rot="R180"/>
-<pinref part="R1" gate="G$1" pin="2"/>
 </segment>
 <segment>
@@
 </segment>
 <segment>
-<pinref part="U$3" gate="G$1" pin="TXD"/>
-<wire x1="76.2" y1="58.42" x2="76.2" y2="66.04" width="0.1524" layer="91"/>
-<label x="76.2" y="66.04" size="1.778" layer="95" rot="R270"/>
-</segment>
-<segment>
-<pinref part="R1" gate="G$1" pin="1"/>
-<wire x1="2.54" y1="83.82" x2="-7.62" y2="83.82" width="0.1524" layer="91"/>
-<label x="-7.62" y="83.82" size="1.778" layer="95"/>
+<pinref part="U$1" gate="G$1" pin="SCK"/>
+<wire x1="40.64" y1="50.8" x2="30.48" y2="50.8" width="0.1524" layer="91"/>
+<label x="30.48" y="50.8" size="1.778" layer="95"/>
 </segment>
 </net>
@@
 <wire x1="114.3" y1="147.32" x2="114.3" y2="142.24" width="0.1524" layer="91"/>
 </segment>
-<segment>
-<pinref part="R2" gate="G$1" pin="1"/>
-<wire x1="-12.7" y1="127" x2="-20.32" y2="127" width="0.1524" layer="91"/>
-<label x="-20.32" y="127" size="1.778" layer="95"/>
-</segment>
-<segment>
-<pinref part="R2" gate="G$1" pin="2"/>
-<wire x1="-2.54" y1="127" x2="5.08" y2="127" width="0.1524" layer="91"/>
-<label x="0" y="127" size="1.778" layer="95"/>
-</segment>
 </net>
