File: files/w20/clock-controller/clock-controller.sch (EAGLE design)
At the start: 12 parts, among them IC1 ATTINY44-SSU

Commit message: fix boards
Connections:
- removed net SCK: U$1.SCK
- net SCL: now also U$1.SCK
Changed lines of the file:
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@@
-</segment>
-</net>
-<net name="SCK" class="0">
-<segment>
-<pinref part="U$1" gate="G$1" pin="SCK"/>
-<wire x1="53.34" y1="17.78" x2="40.64" y2="17.78" width="0.1524" layer="91"/>
-<label x="40.64" y="17.78" size="1.778" layer="95"/>
 </segment>
 </net>
@@
 <label x="132.08" y="43.18" size="1.778" layer="95"/>
 </segment>
+<segment>
+<pinref part="U$1" gate="G$1" pin="SCK"/>
+<wire x1="53.34" y1="17.78" x2="45.72" y2="17.78" width="0.1524" layer="91"/>
+<label x="40.64" y="17.78" size="1.778" layer="95"/>
+<wire x1="43.18" y1="17.78" x2="40.64" y2="17.78" width="0.1524" layer="91"/>
+<wire x1="43.18" y1="17.78" x2="45.72" y2="17.78" width="0.1524" layer="91"/>
+</segment>
 </net>
